File: hardware/pcb/PCB.kicad_pcb (KiCad board)
At the start: 2 copper layers, 53 x 93 mm, 44 parts, among them J1 USB_A, J2 AudioJack3, J3 USB_B_Micro, Q1 BSS138, Q2 S8050, Q3 S8050, SW1 SW_RESET, SW2 S4_SW, U1 ESP32-S3-WROOM-1, U2 LM3525M-H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

Commit message: pcb tweaks
Parts:
- moved R1 13.4 mm to (145.5, 105.1), turned to 180 degrees
- moved C3 9.07 mm to (145.5, 102.2), turned to 0 degrees
- moved R12 7.43 mm to (145.5, 108.0)
- moved D3 7.42 mm to (150.2, 108.0)
- moved C2 6.25 mm to (145.5, 99.2), turned to 180 degrees
- moved Q1 0.50 mm to (135.8, 92.8)
- moved SW1 0.50 mm to (145.5, 94.0), turned to 0 degrees
- moved R4 0.25 mm to (129.5, 92.0)
Routing:
- net Earth: track 149.8 -> 142.2 mm, vias 26 -> 25
- net CHIP_PU: track 88.1 -> 91.2 mm
- net Net-(Q1-Pad2): track 22.9 -> 23.4 mm

Commit message: tweaks
Parts:
- U5: footprint Package_TO_SOT_SMD:SOT-223-3_TabPin2 -> Package_TO_SOT_SMD:SOT-223
- moved C1 9.50 mm to (109.8, 161.0), turned to 0 degrees
- moved R7 4.01 mm to (125.3, 139.6)
- moved C9 3.36 mm to (116.2, 156.0)
- moved R8 2.92 mm to (117.1, 133.5)
- moved U2 2.85 mm to (109.8, 155.8)
- moved R2 1.31 mm to (132.4, 105.2)
- moved R3 0.96 mm to (106.2, 151.0), turned to 180 degrees
- moved C13 0.20 mm to (112.1, 133.5)
- moved U5 0.10 mm to (106.0, 133.5)
Routing:
- net Earth: track 142.2 -> 129.6 mm
- net Net-(R7-Pad2): track 8.44 -> 4.38 mm
- net VBUS: track 153.3 -> 150.7 mm
- net Net-(Q1-Pad2): track 23.4 -> 24.4 mm
- net S4_EN: track 3.56 -> 2.73 mm
- net Net-(Q2-Pad1): track 26.4 -> 25.6 mm
- net Net-(R6-Pad2): track 63.2 -> 64.0 mm
- net Net-(Q3-Pad1): track 12.6 -> 13.2 mm
